Commit message: moving inertial macros to main file

File: batmobile/urdf/batmobile.urdf.xacro (robot description, xacro)
@@ -18,5 +18,4 @@
         </visual>
     </xacro:macro>
-    <xacro:property name="default3d" value="0 0 0"/>
     <xacro:macro name="joint" params="name type parent child axisxyz:=${default3d} originxyz:=${default3d} originrpy:=${default3d}">
         <joint name="${name}" type="${type}">
@@ -35,5 +34,5 @@
                 <material name="blue" />
             </xacro:collision_visual>
-            <xacro:inertial_cylinder mass="2.5" length="0.05" radius="0.1" />
+            <xacro:inertial mass="2.5" ixx="${(1/12) * 2.5 * (3*.1*.1 + 0.05*0.05)}" iyy="${(1/12) * 2.5 * (3*.1*.1 + 0.05*0.05)}" izz="${(1/2) * 2.5 * (.1*.1)}"/>
         </link>
         <xacro:gazebo_material color="Gazebo/Blue" reference="${prefix}_wheel_link" />
@@ -49,12 +48,10 @@
         </visual>
         <collision>
-            <origin xyz="0.0 0.0 0.0" rpy="0. -0.1 0.0" />
+            <origin xyz="0.0 0.0 0.02" rpy="0. -0.15 0.0" />
             <geometry>
                 <box size=".41 .16 .1" />
             </geometry>
         </collision>
-        <xacro:inertial_box mass="10" x=".41" y=".16" z=".1">
-            <origin xyz="0.0 0.0 0.0" rpy="0. -0.05 0.0" />
-    </xacro:inertial_box>
+        <xacro:inertial mass="10" originrpy="0. -0.05 0.0" ixx="${(1/12) * 10 * (.16*.16+.1*.1)}" iyy="${(1/12) * 10 * (.41*.41+.1*.1)}" izz="${(1/12) * 10 * (.41*.41+.16*.16)}"/>
     </link>
     <xacro:wheel_link prefix="left" />
@@ -67,5 +64,5 @@
             <material name="red" />
         </xacro:collision_visual>
-        <xacro:inertial_sphere mass="0.1" radius="0.06"/>
+        <xacro:inertial mass="0.1" ixx="${(2/5) * 0.1*0.06*0.06}" iyy="${(2/5)*0.1*0.06*0.06}" izz="${(2/5)*0.1*0.06*0.06}"/>
     </link>
     <xacro:gazebo_material color="Gazebo/Blue" reference="caster_wheel_link" />

File: batmobile/urdf/inertial_macros.xacro (robot description, xacro)
@@ -1,7 +1,8 @@
 <?xml version="1.0"?>
 <robot xmlns:xacro="http://www.ros.org/wiki/xacro">
-    <xacro:macro name="inertial" params="mass ixx iyy izz origin*">
+    <xacro:property name="default3d" value="0 0 0"/>
+    <xacro:macro name="inertial" params="mass ixx iyy izz originrpy:=${default3d}">
         <inertial>
-            <xacro:insert_block name="origin" />
+            <origin rpy="${originrpy}" />
             <mass value="${mass}" />
             <inertia ixx="${ixx}" ixy="0.0" ixz="0.0" iyy="${iyy}" iyz="0.0" izz="${izz}" />
@@ -11,6 +12,6 @@
         <xacro:inertial mass="${mass}" ixx="${(2/5) * mass*radius*radius}" iyy="${(2/5)*mass*radius*radius}" izz="${(2/5)*mass*radius*radius}" />
     </xacro:macro>
-    <xacro:macro name="inertial_box" params="mass x y z *origin">
-        <xacro:inertial mass="${mass}" ixx="${(1/12) * mass * (y*y+z*z)}" iyy="${(1/12) * mass * (x*x+z*z)}" izz="${(1/12) * mass * (x*x+y*y)}" />
+    <xacro:macro name="inertial_box" params="mass x y z originrpy">
+        <xacro:inertial mass="${mass}" ixx="${(1/12) * mass * (y*y+z*z)}" iyy="${(1/12) * mass * (x*x+z*z)}" izz="${(1/12) * mass * (x*x+y*y)}" originrpy="${originrpy}"/>
     </xacro:macro>
     <xacro:macro name="inertial_cylinder" params="mass length radius">

Commit message: replaced include

File: batmobile/urdf/batmobile.urdf.xacro (robot description, xacro)
@@ -2,6 +2,13 @@
 <robot xmlns:xacro="http://www.ros.org/wiki/xacro" name="batmobile">
     <xacro:include filename="materials.xacro" />
-    <xacro:include filename="inertial_macros.xacro" />
     <xacro:include filename="gazebo_control.xacro" />
+    <xacro:property name="default3d" value="0 0 0"/>
+    <xacro:macro name="inertial" params="mass ixx iyy izz originrpy:=${default3d}">
+        <inertial>
+            <origin rpy="${originrpy}" />
+            <mass value="${mass}" />
+            <inertia ixx="${ixx}" ixy="0.0" ixz="0.0" iyy="${iyy}" iyz="0.0" izz="${izz}" />
+        </inertial>
+    </xacro:macro> <!-- from include inertial_macros -->
     <xacro:macro name="gazebo_material" params="color reference">
         <gazebo reference="${reference}">
