Commit message: broke down inertial macros

File: batmobile/urdf/batmobile.urdf (robot description, URDF)
Before this commit: robot batmobile, 5 links, 4 joints
Links:
- removed link world_link
- added link base_link
- added link imu_link; collision box size=0.03 0.03 0.03; visual box size=0.03 0.03 0.03
- link root_link: geometry collision box size=.41 .16 .1; visual mesh filename=package://batmobile/meshes/chassis.dae scale=0.9 0.5 0.5
Joints:
- added joint imu_joint: type fixed, parent root_link, child imu_link, origin xyz=.205 0 .055 rpy=0 0 0, axis 0 0 0
- joint base_joint: axis 1 1 1 -> 0 0 0; parent world_link -> base_link; type continuous -> fixed
- joint caster_wheel_joint: axis 1 0 0 -> 0 0 0; type continuous -> fixed

File: batmobile/urdf/batmobile.urdf.xacro (robot description, xacro)
@@ -4,7 +4,4 @@
     <xacro:include filename="inertial_macros.xacro" />
     <xacro:include filename="gazebo_control.xacro" />
-    <xacro:property name="chassis_length" value=".41" />
-    <xacro:property name="chassis_width" value=".16" />
-    <xacro:property name="chassis_height" value=".1" />
     <xacro:macro name="gazebo_material" params="color reference">
         <gazebo reference="${reference}">
@@ -43,11 +40,10 @@
         <xacro:joint name="${prefix}_wheel_joint" type="continuous" parent="root_link" child="${prefix}_wheel_link" axisxyz="0 0 ${reflect}" originxyz="-0.05 ${reflect*0.125} 0" originrpy="${-1 * reflect * pi/2} 0 0"/>
     </xacro:macro>
-    <link name="world_link" />
+    <link name="base_link" />
     <link name="root_link">
         <visual>
-            <origin xyz="0.0 0.0 0.02" rpy="0. -0.1 0.0" />
+            <origin xyz="0.0 0.0 0.02" rpy="0. -0.15 0.0" />
             <geometry>
                 <mesh filename="package://batmobile/meshes/chassis.dae" scale="0.9 0.5 0.5" />
-                <!-- <box size="${chassis_length} ${chassis_width} ${chassis_height}" /> -->
             </geometry>
         </visual>
@@ -55,10 +51,10 @@
             <origin xyz="0.0 0.0 0.0" rpy="0. -0.1 0.0" />
             <geometry>
-                <box size="${chassis_length} ${chassis_width} ${chassis_height}" />
+                <box size=".41 .16 .1" />
             </geometry>
         </collision>
-        <xacro:inertial_box mass="10" x="${chassis_length}" y="${chassis_width}" z="${chassis_height}">
+        <xacro:inertial_box mass="10" x=".41" y=".16" z=".1">
             <origin xyz="0.0 0.0 0.0" rpy="0. -0.05 0.0" />
-    </xacro:inertial_box> <!-- can reduce origin since it's just 1 -->
+    </xacro:inertial_box>
     </link>
     <xacro:wheel_link prefix="left" />
@@ -74,5 +70,15 @@
     </link>
     <xacro:gazebo_material color="Gazebo/Blue" reference="caster_wheel_link" />
-    <xacro:joint name="base_joint" originxyz="0 0 .1" child="root_link" parent="world_link" type="fixed"/>
+    <xacro:joint name="base_joint" originxyz="0 0 .1" child="root_link" parent="base_link" type="fixed"/>
     <xacro:joint name="caster_wheel_joint" type="fixed" parent="root_link" child="caster_wheel_link" originxyz="${0.2-0.03} 0.0 -0.03" />
+    <link name="imu_link">
+        <xacro:collision_visual>
+            <geometry>
+                <box size="0.03 0.03 0.03" />
+                <origin xyz="0 0 ${sin(0.15)*.4}"/>
+            </geometry>
+            <material name="green"/>
+        </xacro:collision_visual>
+    </link>
+    <xacro:joint name="imu_joint" type="fixed" parent="root_link" child="imu_link"  originxyz=".205 0 .055" />
 </robot>

File: batmobile/urdf/gazebo_control.xacro (robot description, xacro)
@@ -12,3 +12,13 @@
         </plugin>
     </gazebo>
+    <gazebo>
+        <plugin name="imu_plugin" filename="libgazebo_ros_imu.so">
+          <alwaysOn>true</alwaysOn>
+          <bodyName>imu_link</bodyName>
+          <topicName>imu</topicName>
+          <serviceName>imu_service</serviceName>
+          <gaussianNoise>0.0</gaussianNoise>
+          <updateRate>20.0</updateRate>
+        </plugin>
+      </gazebo>
 </robot>

File: batmobile/urdf/inertial_macros.xacro (robot description, xacro)
@@ -1,28 +1,19 @@
 <?xml version="1.0"?>
 <robot xmlns:xacro="http://www.ros.org/wiki/xacro">
- <xacro:macro name="inertial_sphere" params="mass radius">
-     <inertial>
-         <mass value="${mass}"/>
-         <inertia ixx="${(2/5) * mass*radius*radius}" ixy="0.0" ixz="0.0"
-         iyy="${(2/5)*mass*radius*radius}" iyz="0.0"
-         izz="${(2/5)*mass*radius*radius}"/>
-     </inertial>
- </xacro:macro>
- <xacro:macro name="inertial_box" params="mass x y z *origin">
-    <inertial>
-        <xacro:insert_block name="origin"/>
-        <mass value="${mass}" />
-        <inertia ixx="${(1/12) * mass * (y*y+z*z)}" ixy="0.0" ixz="0.0"
-                iyy="${(1/12) * mass * (x*x+z*z)}" iyz="0.0"
-                izz="${(1/12) * mass * (x*x+y*y)}" />
-    </inertial>
-</xacro:macro>
-<xacro:macro name="inertial_cylinder" params="mass length radius">
-    <inertial>
-        <mass value="${mass}" />
-        <inertia ixx="${(1/12) * mass * (3*radius*radius + length*length)}" ixy="0.0" ixz="0.0"
-                iyy="${(1/12) * mass * (3*radius*radius + length*length)}" iyz="0.0"
-                izz="${(1/2) * mass * (radius*radius)}" />
-    </inertial>
-</xacro:macro>
+    <xacro:macro name="inertial" params="mass ixx iyy izz origin*">
+        <inertial>
+            <xacro:insert_block name="origin" />
+            <mass value="${mass}" />
+            <inertia ixx="${ixx}" ixy="0.0" ixz="0.0" iyy="${iyy}" iyz="0.0" izz="${izz}" />
+        </inertial>
+    </xacro:macro>
+    <xacro:macro name="inertial_sphere" params="mass radius">
+        <xacro:inertial mass="${mass}" ixx="${(2/5) * mass*radius*radius}" iyy="${(2/5)*mass*radius*radius}" izz="${(2/5)*mass*radius*radius}" />
+    </xacro:macro>
+    <xacro:macro name="inertial_box" params="mass x y z *origin">
+        <xacro:inertial mass="${mass}" ixx="${(1/12) * mass * (y*y+z*z)}" iyy="${(1/12) * mass * (x*x+z*z)}" izz="${(1/12) * mass * (x*x+y*y)}" />
+    </xacro:macro>
+    <xacro:macro name="inertial_cylinder" params="mass length radius">
+        <xacro:inertial mass="${mass}" ixx="${(1/12) * mass * (3*radius*radius + length*length)}" iyy="${(1/12) * mass * (3*radius*radius + length*length)}" izz="${(1/2) * mass * (radius*radius)}" />
+    </xacro:macro>
 </robot>

Commit message: added 1 more joint to caster wheel

File: batmobile/urdf/batmobile.urdf (robot description, URDF)
Before this commit: robot batmobile, 6 links, 5 joints
Links:
- added link caster_wheel_holder; collision cylinder length=0.01 radius=0.001; visual cylinder length=0.01 radius=0.001
Joints:
- added joint caster_wheel_holder_joint: type continuous, parent root_link, child caster_wheel_holder, origin xyz=0.17 0.0 -0.03 rpy=0 0 0, axis 0 0 1
- joint caster_wheel_joint: axis 0 0 0 -> 0 1 0; type fixed -> continuous

File: batmobile/urdf/batmobile.urdf.xacro (robot description, xacro)
@@ -2,7 +2,5 @@
 <robot xmlns:xacro="http://www.ros.org/wiki/xacro" name="batmobile">
     <xacro:macro name="material_color" params="name rgba">
-        <material name="${name}">
-            <color rgba="${rgba}" />
-        </material>
+        <material name="${name}"><color rgba="${rgba}" /></material>
     </xacro:macro>
     <xacro:material_color name="blue" rgba="0.0 0.0 0.8 1.0" />
@@ -73,6 +71,5 @@
         <xacro:joint name="${prefix}_wheel_joint" type="continuous" parent="root_link" child="${prefix}_wheel_link" axisxyz="0 0 ${reflect}" originxyz="-0.05 ${reflect*0.125} 0" originrpy="${-1 * reflect * pi/2} 0 0" />
     </xacro:macro>
-    <link name="base_link" />
-    <link name="root_link">
+    <link name="base_link" /><link name="root_link">
         <visual>
             <origin xyz="0.0 0.0 0.02" rpy="0. -0.15 0.0" />
@@ -100,12 +97,20 @@
         <xacro:inertial mass="0.1" ixx="${(2/5) * 0.1*0.06*0.06}" iyy="${(2/5)*0.1*0.06*0.06}" izz="${(2/5)*0.1*0.06*0.06}" />
     </link>
+    <link name="caster_wheel_holder">
+        <xacro:collision_visual>
+            <geometry>
+                <cylinder length="0.01" radius="0.001" />
+            </geometry>
+            <material name="green"/>
+        </xacro:collision_visual>
+    </link>
     <xacro:gazebo_material color="Gazebo/Blue" reference="caster_wheel_link" />
     <xacro:joint name="base_joint" originxyz="0 0 .1" child="root_link" parent="base_link" type="fixed" />
-    <xacro:joint name="caster_wheel_joint" type="fixed" parent="root_link" child="caster_wheel_link" originxyz="${0.2-0.03} 0.0 -0.03" />
+    <xacro:joint name="caster_wheel_holder_joint" type="continuous" axisxyz="0 0 1" parent="root_link" child="caster_wheel_holder" originxyz="${0.2-0.03} 0.0 -0.03" />
+    <xacro:joint name="caster_wheel_joint" type="continuous" axisxyz="0 1 0" parent="root_link" child="caster_wheel_link" originxyz="${0.2-0.03} 0.0 -0.03" />
     <link name="imu_link">
         <xacro:collision_visual>
             <geometry>
-                <box size="0.03 0.03 0.03" />
-                <origin xyz="0 0 ${sin(0.15)*.4}" />
+                <box size="0.03 0.03 0.03" /><origin xyz="0 0 ${sin(0.15)*.4}" />
             </geometry>
             <material name="green" />
